File: peripherals.kicad_sch (KiCad schematic)
At the start: 33 parts, among them J201 Motor_1, J202 Motor_2, U201 A3901SEJTR-T, U202 ICM-42670-P, U203 NH-B1515RGBA-HF

Commit message: production time
Parts:
- removed J201: Motor_1, Connector_JST:JST_PH_B2B-PH-K_1x02_P2.00mm_Vertical, symbol Connector_Generic:Conn_01x02
- removed J202: Motor_2, Connector_JST:JST_PH_B2B-PH-K_1x02_P2.00mm_Vertical, symbol Connector_Generic:Conn_01x02
- added U205: Motor_1, footprints:CONN-TH_BM02B-SRSS-TB-LF-SN, symbol BM02B-SRSS-TB_(LF)(SN):BM02B-SRSS-TB_(LF)(SN)
- added U206: Motor_2, footprints:CONN-TH_BM02B-SRSS-TB-LF-SN, symbol BM02B-SRSS-TB_(LF)(SN):BM02B-SRSS-TB_(LF)(SN)
- C204: footprint Capacitor_SMD:C_0402_1005Metric -> Capacitor_SMD:C_0603_1608Metric
- JP201, JP202: footprint (none) -> Jumper:SolderJumper-2_P1.3mm_Bridged_RoundedPad1.0x1.5mm
- TP201, TP202, TP203, TP204, TP205, TP206, TP207, TP208, TP209, TP210, TP211, TP212, TP213, TP214: footprint (none) -> Connector_Pin:Pin_D1.0mm_L10.0mm
- U204: footprint poka-yoke_txrx:poka-yoke_txrx -> poka-yoke_rxtx:poka-yoke_rxtx
Connections:
- net +3V3: no longer D201.2 (A)
- net GND: now also U205.3, U205.4, U206.3, U206.4
- net INT1: now also TP213.1; no longer TP214.1
- net INT2: now also TP214.1; no longer TP213.1
- net SDI_ESP: now also U204.1 (Rx_In); no longer U204.3 (Tx_Out)
- net SDI_IMU: now also U204.2 (Tx_In); no longer U204.1 (Rx_In)
- net SDO_ESP: now also U204.3 (Tx_Out); no longer U204.4 (Rx_Out)
- net SDO_IMU: now also U204.4 (Rx_Out); no longer U204.2 (Tx_In)
- net at TP205.1, U201.10 (OUT1): now also U205.1
- net at TP206.1, U201.9 (OUT2): now also U205.2
- net at TP207.1, U201.7 (OUT3): now also U206.1
- net at TP208.1, U201.6 (OUT4): now also U206.2
- net IMU_FSYNC: no longer names the net of U202.7 (FSYNC)
- new net +5V: D201.2 (A)
- no-connect marks 0 -> 1
Other:
- moved on the sheet: C204, JP201, R204, R205, TP201, TP202, TP203, TP204, TP205, TP206, TP207, TP208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
