File: swarm-pcb.kicad_pcb (KiCad board)
At the start: 2 copper layers, 60 parts, among them J101 Conn_ARM_SWD_TagConnect_TC2030, J201 Motor_1, J202 Motor_2, Q301 CJ3139K, U101 USB-TYPE-C-018, U102 2450AT18A100E, U103 ESP32-S3, U104 TS-1187A-B-A-B, U105 TS-1187A-B-A-B, U201 A3901SEJTR-T, U202 ICM-42670-P, U203 NH-B1515RGBA-HF, U301 TLV62569DRL, U302 TP4065, X101 TZ1269D

Commit message: production time
Parts:
- removed C111: 1pF, Capacitor_SMD:C_0402_1005Metric
- removed C117: 12pF/10V, Capacitor_SMD:C_0603_1608Metric
- removed D302: WHITE, LED_SMD:LED_0603_1608Metric
- removed J101: Conn_ARM_SWD_TagConnect_TC2030, Connector:Tag-Connect_TC2030-IDC-FP_2x03_P1.27mm_Vertical
- removed J201: Motor_1, Connector_JST:JST_PH_B2B-PH-K_1x02_P2.00mm_Vertical
- removed J202: Motor_2, Connector_JST:JST_PH_B2B-PH-K_1x02_P2.00mm_Vertical
- removed L102: 3.9nH, Inductor_SMD:L_0402_1005Metric
- removed R303: 1kΩ, Resistor_SMD:R_0402_1005Metric
- added C114: 0.1uF/10V, Capacitor_SMD:C_0402_1005Metric, F.Cu at (75.2, 129.5)
- added C115: 12pF/10V, Capacitor_SMD:C_0603_1608Metric, F.Cu at (101.5, 130.7)
- added C204: 10uF, Capacitor_SMD:C_0603_1608Metric, F.Cu at (82.0, 136.4)
- added JP201: SJ_MOTOR_3V3, Jumper:SolderJumper-2_P1.3mm_Bridged_RoundedPad1.0x1.5mm, F.Cu at (85.2, 136.4)
- added JP202: SJ_IMU_3V3, Jumper:SolderJumper-2_P1.3mm_Bridged_RoundedPad1.0x1.5mm, F.Cu at (79.1, 120.1)
- added R104: 22Ω, Resistor_SMD:R_0402_1005Metric, F.Cu at (99.0, 129.5)
- added R105: 0Ω, Resistor_SMD:R_0402_1005Metric, F.Cu at (105.5, 125.0)
- added R106: 0Ω, Resistor_SMD:R_0402_1005Metric, F.Cu at (102.2, 125.0)
- added REF**: test from isaac, footprints:test from isaac, B.Cu at (99.7, 114.5)
- added TP101: TP_5V0, Connector_Pin:Pin_D1.0mm_L10.0mm, F.Cu at (70.5, 132.7)
- added TP102: TP_XTAL_P, Connector_Pin:Pin_D1.0mm_L10.0mm, F.Cu at (102.0, 133.8)
- added TP103: TP_BOOT, Connector_Pin:Pin_D1.0mm_L10.0mm, F.Cu at (95.2, 115.5)
- added TP104: TP_RESET, Connector_Pin:Pin_D1.0mm_L10.0mm, F.Cu at (84.2, 109.4)
- added TP201: TP_MOTOR_CTRL_2, Connector_Pin:Pin_D1.0mm_L10.0mm, F.Cu at (100.2, 139.3)
- added TP202: TP_MOTOR_CTRL_1, Connector_Pin:Pin_D1.0mm_L10.0mm, F.Cu at (100.2, 136.2)
- added TP203: TP_MOTOR_CTRL_4, Connector_Pin:Pin_D1.0mm_L10.0mm, F.Cu at (100.2, 145.4)
- added TP204: TP_MOTOR_CTRL_3, Connector_Pin:Pin_D1.0mm_L10.0mm, F.Cu at (100.2, 142.4)
- added TP205: TP_MOTOR_1_1, Connector_Pin:Pin_D1.0mm_L10.0mm, F.Cu at (93.4, 139.2)
- added TP206: TP_MOTOR_1_2, Connector_Pin:Pin_D1.0mm_L10.0mm, F.Cu at (90.3, 139.2)
- added TP207: TP_MOTOR_2_1, Connector_Pin:Pin_D1.0mm_L10.0mm, F.Cu at (87.3, 139.2)
- added TP208: TP_MOTOR_2_2, Connector_Pin:Pin_D1.0mm_L10.0mm, F.Cu at (84.3, 139.2)
- added TP209: TP_SDO_IMU, Connector_Pin:Pin_D1.0mm_L10.0mm, F.Cu at (75.5, 111.2)
- added TP210: TP_SDI_IMU, Connector_Pin:Pin_D1.0mm_L10.0mm, F.Cu at (72.4, 111.2)
- added TP211: TP_CS, Connector_Pin:Pin_D1.0mm_L10.0mm, F.Cu at (81.5, 111.3)
- added TP212: TP_SCLK, Connector_Pin:Pin_D1.0mm_L10.0mm, F.Cu at (78.5, 111.2)
- added TP213: TP_INT1, Connector_Pin:Pin_D1.0mm_L10.0mm, F.Cu at (70.3, 113.5)
- added TP214: TP_INT2, Connector_Pin:Pin_D1.0mm_L10.0mm, F.Cu at (81.8, 121.2)
- added TP301: TP_3V3, Connector_Pin:Pin_D1.0mm_L10.0mm, F.Cu at (87.3, 130.6)
- added TP302: TP_VBUS, Connector_Pin:Pin_D1.0mm_L10.0mm, F.Cu at (77.9, 134.7)
- added TP303: TP_VBATT, Connector_Pin:Pin_D1.0mm_L10.0mm, F.Cu at (71.1, 141.9)
- added TP304: TP_BATT_STAT, Connector_Pin:Pin_D1.0mm_L10.0mm, F.Cu at (68.2, 141.2)
- added TP305: TP_BATT_PROG, Connector_Pin:Pin_D1.0mm_L10.0mm, F.Cu at (68.2, 138.1)
- added TP306: TP_FB_3V3, Connector_Pin:Pin_D1.0mm_L10.0mm, F.Cu at (78.2, 128.5)
- added TP307: TP_BUCK_GND, Connector_Pin:Pin_D1.0mm_L10.0mm, F.Cu at (75.2, 132.2)
- added U205: Motor_1, footprints:CONN-TH_BM02B-SRSS-TB-LF-SN, F.Cu at (91.5, 143.9)
- added U206: Motor_2, footprints:CONN-TH_BM02B-SRSS-TB-LF-SN, F.Cu at (85.9, 143.9)
- added U303: BATT, footprints:CONN-TH_BM02B-SRSS-TB-LF-SN, F.Cu at (76.0, 143.1)
- added kibuzzard-672F6F41: G***, kibuzzard-672F6F41, F.Cu at (70.9, 116.5)
- added kibuzzard-672F6FA2: G***, kibuzzard-672F6FA2, F.Cu at (81.5, 142.5)
- added kibuzzard-672F6FAB: G***, kibuzzard-672F6FAB, F.Cu at (96.1, 142.5)
- added kibuzzard-672F6FBA: G***, kibuzzard-672F6FBA, F.Cu at (70.1, 144.5)
- added kibuzzard-672F6FFE: G***, kibuzzard-672F6FFE, F.Cu at (87.3, 133.2)
- added kibuzzard-672F7049: G***, kibuzzard-672F7049, F.Cu at (90.7, 114.1)
- added kibuzzard-672F7060: G***, kibuzzard-672F7060, F.Cu at (103.7, 112.3)
- added kibuzzard-672F708E: G***, kibuzzard-672F708E, F.Cu at (78.5, 123.0)
- added kibuzzard-673054F1: G***, kibuzzard-673054F1, B.Cu at (83.0, 113.6)
- added kibuzzard-67305501: G***, kibuzzard-67305501, B.Cu at (80.8, 114.6)
- added kibuzzard-67305511: G***, kibuzzard-67305511, B.Cu at (78.7, 115.5)
- added kibuzzard-6730551F: G***, kibuzzard-6730551F, B.Cu at (76.0, 115.5)
- added kibuzzard-6730552C: G***, kibuzzard-6730552C, B.Cu at (73.0, 116.2)
- added kibuzzard-67305534: G***, kibuzzard-67305534, B.Cu at (87.3, 112.8)
- added kibuzzard-67305547: G***, kibuzzard-67305547, B.Cu at (84.8, 124.0)
- added kibuzzard-67305558: G***, kibuzzard-67305558, B.Cu at (81.8, 132.0)
- added kibuzzard-6730556D: G***, kibuzzard-6730556D, B.Cu at (90.1, 132.8)
- added kibuzzard-67305590: G***, kibuzzard-67305590, B.Cu at (96.7, 133.7)
- added kibuzzard-6730559C: G***, kibuzzard-6730559C, B.Cu at (95.5, 136.2)
- added kibuzzard-673055BA: G***, kibuzzard-673055BA, B.Cu at (95.5, 145.5)
- added kibuzzard-673055CB: G***, kibuzzard-673055CB, B.Cu at (93.4, 141.8)
- added kibuzzard-673055DA: G***, kibuzzard-673055DA, B.Cu at (84.0, 141.8)
- added kibuzzard-673055F3: G***, kibuzzard-673055F3, B.Cu at (77.0, 130.8)
- added kibuzzard-673055FE: G***, kibuzzard-673055FE, B.Cu at (78.0, 136.8)
- added kibuzzard-6730560C: G***, kibuzzard-6730560C, B.Cu at (69.4, 135.4)
- added kibuzzard-6730561B: G***, kibuzzard-6730561B, B.Cu at (75.4, 139.3)
- added kibuzzard-6730566E: G***, kibuzzard-6730566E, B.Cu at (100.3, 121.1)
- added kibuzzard-6730568D: G***, kibuzzard-6730568D, B.Cu at (93.8, 118.5)
- added kibuzzard-673056FB: G***, kibuzzard-673056FB, B.Cu at (88.8, 126.8)
- added kibuzzard-67305712: G***, kibuzzard-67305712, B.Cu at (98.6, 124.3)
- added kibuzzard-67305722: G***, kibuzzard-67305722, B.Cu at (95.2, 128.6)
- moved Q301 74.4 mm to (74.7, 139.6)
- moved R304 74.4 mm to (70.5, 135.8), turned to 180 degrees
- moved R302 74.0 mm to (72.4, 135.8), turned to 180 degrees
- moved U302 73.9 mm to (71.7, 138.3), turned to -90 degrees
- moved R101 70.2 mm to (75.4, 128.1), turned to 180 degrees
- moved C303 69.0 mm to (74.5, 136.3), turned to 90 degrees
- moved L301 69.0 mm to (82.1, 134.1), turned to 180 degrees
- moved D301 67.8 mm to (77.0, 139.1), turned to -90 degrees
- moved R102 67.3 mm to (75.1, 123.8), turned to 90 degrees
- moved U301 67.2 mm to (81.1, 131.6)
- moved C305 64.8 mm to (81.1, 130.0)
- moved U101 63.8 mm to (71.1, 126.2), turned to -90 degrees
- moved C304 62.1 mm to (79.0, 131.6), turned to 90 degrees
- moved U103 61.1 mm to (93.7, 127.0), turned to -135 degrees
- moved D201 60.7 mm to (71.0, 119.7)
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Connections:
- C105 pad 1: /VDD_SPI -> +3V3
- C107 pad 1: /VDD_SPI -> +3V3
- C112 pad 1: Net-(C112-Pad1) -> /RESET
- C201 pad 1: +3V3 -> Net-(JP202-A)
- C202 pad 1: +3V3 -> Net-(JP202-A)
- D201 pad 2: +3V3 -> +5V
- R103 pad 2: Net-(C112-Pad1) -> /RESET
- R201 pad 1: /peripherals/BLUE -> BLUE
- R202 pad 2: /peripherals/GREEN -> GREEN
- R203 pad 2: /peripherals/RED -> RED
- R204 pad 2: /peripherals/SDO_ESP -> SDO_ESP
- R205 pad 2: /peripherals/SDI_ESP -> SDI_ESP
- U103 pad 10: unconnected-(U103-GPIO5-Pad10) -> GREEN
- U103 pad 15: /CS -> CS
- U103 pad 16: /SDI_ESP -> SDI_ESP
- U103 pad 17: /SCLK -> SCLK
- U103 pad 18: /SDO_ESP -> SDO_ESP
- U103 pad 23: unconnected-(U103-GPIO17-Pad23) -> INT2
- U103 pad 24: unconnected-(U103-GPIO18-Pad24) -> INT1
- U103 pad 29: /VDD_SPI -> +3V3
- U103 pad 38: unconnected-(U103-GPIO33-Pad38) -> MOTOR_CTRL_4
- U103 pad 39: unconnected-(U103-GPIO34-Pad39) -> MOTOR_CTRL_3
- U103 pad 40: unconnected-(U103-GPIO35-Pad40) -> MOTOR_CTRL_2
- U103 pad 41: unconnected-(U103-GPIO36-Pad41) -> MOTOR_CTRL_1
- U103 pad 8: unconnected-(U103-GPIO3-Pad8) -> BLUE
- U103 pad 9: unconnected-(U103-GPIO4-Pad9) -> RED
- U201 pad 1: /peripherals/MOTOR_CTRL_1 -> MOTOR_CTRL_1
- U201 pad 2: /peripherals/MOTOR_CTRL_2 -> MOTOR_CTRL_2
- U201 pad 4: /peripherals/MOTOR_CTRL_3 -> MOTOR_CTRL_3
- U201 pad 5: /peripherals/MOTOR_CTRL_4 -> MOTOR_CTRL_4
- U201 pad 8: +3V3 -> Net-(JP201-A)
- U202 pad 12: /peripherals/CS -> CS
- U202 pad 13: /peripherals/SCLK -> SCLK
- U202 pad 4: /peripherals/INT1 -> INT1
- U202 pad 7: /peripherals/IMU_FSYNC -> unconnected-(U202-FSYNC-Pad7)
- U202 pad 8: +3V3 -> Net-(JP202-A)
- U202 pad 9: /peripherals/INT2 -> INT2
- U204 pad 1: /peripherals/SDI_IMU -> SDI_ESP
- U204 pad 2: /peripherals/SDO_IMU -> /peripherals/SDI_IMU
- U204 pad 3: /peripherals/SDI_ESP -> SDO_ESP
- U204 pad 4: /peripherals/SDO_ESP -> /peripherals/SDO_IMU
- X101 pad 1: /XTAL_N -> Net-(C115-Pad1)
- X101 pad 3: /XTAL_P -> /XTAL_N
Routing:
- net +3V3: track 0.00 -> 110.1 mm, vias 0 -> 9
- net INT1: track 0.00 -> 36.4 mm
- net +5V: track 0.00 -> 36.0 mm
- net /RESET: track 0.00 -> 34.8 mm
- net MOTOR_CTRL_4: track 0.00 -> 25.0 mm, vias 0 -> 1
- net CS: track 0.00 -> 23.6 mm, vias 0 -> 3
- net SCLK: track 0.00 -> 23.2 mm, vias 0 -> 3
- net MOTOR_CTRL_3: track 0.00 -> 20.9 mm, vias 0 -> 1
- net MOTOR_CTRL_2: track 0.00 -> 20.0 mm, vias 0 -> 1
- net /USB_N: track 0.00 -> 19.8 mm
- net /USB_P: track 0.00 -> 19.4 mm
- net /peripherals/SDO_IMU: track 0.00 -> 17.3 mm
- net INT2: track 0.00 -> 16.7 mm
- net MOTOR_CTRL_1: track 0.00 -> 14.3 mm, vias 0 -> 1
- net /BOOT: track 0.00 -> 13.4 mm
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- added copper zone on B.Cu, net GND
- added copper zone on F.Cu, net GND
- added copper zone on In1.Cu, net GND
- added copper zone on In2.Cu, net GND
Other:
- board outline added: 45 x 40 mm
- copper layers 2 -> 4
- board text added: "JLC04101H-7628 Stackup L1/L2 | trace spacing | trace to copper 50Ω single ended: / 0.127 => 0.2380 90Ω diff pair: 0.127 0.127 => 0.1748 L1/L3 90Ω diff pair: 0.127 0.127 => 0.1377"
- board text added: "TODO: need battery polarity"
