File: swarm-pcb.kicad_sch (KiCad schematic)
At the start: 32 parts, among them U101 USB-TYPE-C-018, U102 2450AT18A100E, U103 ESP32-S3, U104 TS-1187A-B-A-B, U105 TS-1187A-B-A-B, X101 TZ1269D

Commit message: production time
Parts:
- removed C111: 1pF, Capacitor_SMD:C_0402_1005Metric, symbol Device:C
- removed C117: 12pF/10V, Capacitor_SMD:C_0603_1608Metric, symbol Device:C
- removed L102: 3.9nH, Inductor_SMD:L_0402_1005Metric, symbol Device:L
- removed TP105: TP_GND, symbol Connector:TestPoint
- added C114: 0.1uF/10V, Capacitor_SMD:C_0402_1005Metric, symbol Device:C
- added C115: 12pF/10V, Capacitor_SMD:C_0603_1608Metric, symbol Device:C
- added R104: 22Ω, Resistor_SMD:R_0402_1005Metric, symbol Device:R
- added R105, R106: 0Ω, Resistor_SMD:R_0402_1005Metric, symbol Device:R
- TP101, TP102, TP103, TP104: footprint (none) -> Connector_Pin:Pin_D1.0mm_L10.0mm
Connections:
- net VDD_SPI is gone; now on net +3V3: C105.1, C107.1, U103.29 (VDD_SPI)
- net +5V: now also C114.1
- net BLUE: now also U103.8 (GPIO3)
- net GND: now also C114.2, C115.2
- net GREEN: now also U103.10 (GPIO5)
- net INT1: now also U103.24 (GPIO18)
- net INT2: now also U103.23 (GPIO17)
- net LNA_IN: now also R106.2
- net MOTOR_CTRL_1: now also U103.41 (GPIO36)
- net MOTOR_CTRL_2: now also U103.40 (GPIO35)
- net MOTOR_CTRL_3: now also U103.39 (GPIO34)
- net MOTOR_CTRL_4: now also U103.38 (GPIO33)
- net RED: now also U103.9 (GPIO4)
- net RESET: now also C112.1, R103.2
- net XTAL_N: now also X101.3; no longer X101.1
- net XTAL_P: now also R104.1; no longer TP102.1, X101.3
- net at L103.1: now also R105.2, R106.1
- net at U102.1 (ANT): now also R105.1
- new net: C115.1, R104.2, TP102.1, X101.1
- no-connect marks 22 -> 36
Other:
- note added: "1pF"
- note added: "3.9nH"
- moved on the sheet: C118, TP102, X101
