File: power.kicad_sch (KiCad schematic)
At the start: 22 parts, among them Q301 CJ3139K, U301 TLV62569DRL, U302 TP4065

Commit message: production time
Parts:
- removed D302: WHITE, LED_SMD:LED_0603_1608Metric, symbol Device:LED
- removed R303: 1kΩ, Resistor_SMD:R_0402_1005Metric, symbol Device:R
- added TP307: TP_BUCK_GND, Connector_Pin:Pin_D1.0mm_L10.0mm, symbol Connector:TestPoint
- added U303: BATT, footprints:CONN-TH_BM02B-SRSS-TB-LF-SN, symbol BM02B-SRSS-TB_(LF)(SN):BM02B-SRSS-TB_(LF)(SN)
- R302: now not fitted
- TP301, TP302, TP303, TP304, TP305, TP306: footprint (none) -> Connector_Pin:Pin_D1.0mm_L10.0mm
Connections:
- net +BATT: now also U303.1
- net GND: now also TP307.1, U303.2, U303.3, U303.4
Other:
- moved on the sheet: C303, D301, Q301, R304, TP303, TP304, TP305, U302

Commit message: production
Other:
- note added: "LED would pull down the line automatically."
Changed lines of the file:
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@@
+		)
+	)
+	(text "LED would pull down \nthe line automatically."
+		(exclude_from_sim no)
+		(at 62.992 64.516 0)
+		(effects
+			(font
+				(size 1.27 1.27)
+			)
 		)
 	)
